File: STM32F446RE_subcircuit/STM32F446RE_subcircuit.brd (EAGLE design)
At the start: 88.6 x 55.9 mm, 49 parts, among them IC2 LD117AS33TR, U1 STM32F446RE, X1 MSTBA2, X2 32.768kHz, X3 8MHz

Commit message: remaining changes
Routing:
- added copper zone on layer 1, net HEAT
- added copper zone on layer 16, net HEAT
- removed copper zone on layer 1, net N$13
- removed copper zone on layer 16, net N$14
- removed copper zone on layer 16, net N$15
