File: Breakout board files/AT45DB041ESHNB.sch (EAGLE design)
At the start: 9 parts, among them U1 AT45DB041E-SHN-B

Commit message: Breakout Board Solutions
Parts:
- removed PAD1, PAD2, PAD3, PAD4, PAD5, PAD6, PAD7, PAD8: (no value), ee2parts:PAD-TERMINAL
- added JP1, JP2: (no value), pinhead:PINHD-1X4
Connections:
- removed net N$1: PAD1.P, U1.VCC
- removed net N$2: PAD2.P, U1.SI
- removed net N$3: PAD3.P, U1.SCK
- removed net N$4: PAD4.P, U1.~RESET
- removed net N$5: PAD5.P, U1.~CS
- removed net N$6: PAD6.P, U1.~WP
- removed net N$7: PAD7.P, U1.GND
- removed net N$8: PAD8.P, U1.SO
- new net 1: JP2.1, U1.SI
- new net 2: JP2.2, U1.SCK
- new net 3: JP2.3, U1.~RESET
- new net 4: JP2.4, U1.~CS
- new net 5: JP1.1, U1.~WP
- new net 6: JP1.2, U1.VCC
- new net 7: JP1.3, U1.GND
- new net 8: JP1.4, U1.SO
Changed lines of the file:
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@@
 <?xml version="1.0" encoding="utf-8"?>
 <!DOCTYPE eagle SYSTEM "eagle.dtd">
-<eagle version="8.3.2">
+<eagle version="9.2.0">
 <drawing>
 <settings>
@@
 <layers>
 <layer number="1" name="Top" color="4" fill="1" visible="no" active="no"/>
+<layer number="2" name="Route2" color="1" fill="3" visible="no" active="no"/>
+<layer number="3" name="Route3" color="4" fill="3" visible="no" active="no"/>
+<layer number="4" name="Route4" color="1" fill="4" visible="no" active="no"/>
+<layer number="5" name="Route5" color="4" fill="4" visible="no" active="no"/>
+<layer number="6" name="Route6" color="1" fill="8" visible="no" active="no"/>
+<layer number="7" name="Route7" color="4" fill="8" visible="no" active="no"/>
+<layer number="8" name="Route8" color="1" fill="2" visible="no" active="no"/>
+<layer number="9" name="Route9" color="4" fill="2" visible="no" active="no"/>
+<layer number="10" name="Route10" color="1" fill="7" visible="no" active="no"/>
+<layer number="11" name="Route11" color="4" fill="7" visible="no" active="no"/>
+<layer number="12" name="Route12" color="1" fill="5" visible="no" active="no"/>
+<layer number="13" name="Route13" color="4" fill="5" visible="no" active="no"/>
+<layer number="14" name="Route14" color="1" fill="6" visible="no" active="no"/>
+<layer number="15" name="Route15" color="4" fill="6" visible="no" active="no"/>
 <layer number="16" name="Bottom" color="1" fill="1" visible="no" active="no"/>
 <layer number="17" name="Pads" color="2" fill="1" visible="no" active="no"/>
@@
 <parts>
 <part name="U1" library="AT45DB041E-SHN-B" deviceset="AT45DB041E-SHN-B" device=""/>
-<part name="PAD1" library="ee2parts" deviceset="PAD-TERMINAL" device=""/>
-<part name="PAD2" library="ee2parts" deviceset="PAD-TERMINAL" device=""/>
-<part name="PAD3" library="ee2parts" deviceset="PAD-TERMINAL" device=""/>
-<part name="PAD4" library="ee2parts" deviceset="PAD-TERMINAL" device=""/>
-<part name="PAD5" library="ee2parts" deviceset="PAD-TERMINAL" device=""/>
-<part name="PAD6" library="ee2parts" deviceset="PAD-TERMINAL" device=""/>
-<part name="PAD7" library="ee2parts" deviceset="PAD-TERMINAL" device=""/>
-<part name="PAD8" library="ee2parts" deviceset="PAD-TERMINAL" device=""/>
+<part name="JP1" library="pinhead" library_urn="urn:adsk.eagle:library:325" deviceset="PINHD-1X4" device="" package3d_urn="urn:adsk.eagle:package:22407/2"/>
+<part name="JP2" library="pinhead" library_urn="urn:adsk.eagle:library:325" deviceset="PINHD-1X4" device="" package3d_urn="urn:adsk.eagle:package:22407/2"/>
 </parts>
 <sheets>
@@
 </plain>
 <instances>
-<instance part="U1" gate="A" x="63.5" y="50.8"/>
-<instance part="PAD1" gate="1" x="35.56" y="60.96"/>
-<instance part="PAD2" gate="1" x="35.56" y="55.88"/>
-<instance part="PAD3" gate="1" x="35.56" y="50.8"/>
-<instance part="PAD4" gate="1" x="35.56" y="45.72"/>
-<instance part="PAD5" gate="1" x="35.56" y="40.64"/>
-<instance part="PAD6" gate="1" x="35.56" y="35.56"/>
-<instance part="PAD7" gate="1" x="35.56" y="30.48"/>
-<instance part="PAD8" gate="1" x="91.44" y="58.42" rot="R180"/>
+<instance part="U1" gate="A" x="63.5" y="50.8">
+<attribute name="NAME" x="57.537709375" y="66.0625" size="2.08935" layer="95" ratio="10" rot="SR0"/>
+<attribute name="VALUE" x="59.125740625" y="28.2421" size="2.0854" layer="96" ratio="10" rot="SR0"/>
+</instance>
+<instance part="JP1" gate="A" x="106.68" y="53.34">
+<attribute name="NAME" x="100.33" y="61.595" size="1.778" layer="95"/>
+<attribute name="VALUE" x="100.33" y="45.72" size="1.778" layer="96"/>
+</instance>
+<instance part="JP2" gate="A" x="15.24" y="48.26" rot="R180">
+<attribute name="NAME" x="21.59" y="40.005" size="1.778" layer="95" rot="R180"/>
+<attribute name="VALUE" x="21.59" y="55.88" size="1.778" layer="96" rot="R180"/>
+</instance>
 </instances>
 <busses>
 </busses>
 <nets>
-<net name="N$1" class="0">
+<net name="6" class="0">
 <segment>
 <pinref part="U1" gate="A" pin="VCC"/>
-<pinref part="PAD1" gate="1" pin="P"/>
 <wire x1="45.72" y1="58.42" x2="38.1" y2="58.42" width="0.1524" layer="91"/>
-<wire x1="38.1" y1="58.42" x2="38.1" y2="60.96" width="0.1524" layer="91"/>
-</segment>
-</net>
-<net name="N$2" class="0">
+<label x="40.64" y="58.42" size="1.778" layer="95"/>
+</segment>
+<segment>
+<pinref part="JP1" gate="A" pin="2"/>
+<wire x1="104.14" y1="55.88" x2="93.98" y2="55.88" width="0.1524" layer="91"/>
+<label x="93.98" y="55.88" size="1.778" layer="95"/>
+</segment>
+</net>
+<net name="1" class="0">
 <segment>
 <pinref part="U1" gate="A" pin="SI"/>
-<pinref part="PAD2" gate="1" pin="P"/>
 <wire x1="45.72" y1="53.34" x2="38.1" y2="53.34" width="0.1524" layer="91"/>
-<wire x1="38.1" y1="53.34" x2="38.1" y2="55.88" width="0.1524" layer="91"/>
-</segment>
-</net>
-<net name="N$3" class="0">
+<label x="40.64" y="53.34" size="1.778" layer="95"/>
+</segment>
+<segment>
+<pinref part="JP2" gate="A" pin="1"/>
+<wire x1="17.78" y1="43.18" x2="27.94" y2="43.18" width="0.1524" layer="91"/>
+<label x="22.86" y="43.18" size="1.778" layer="95"/>
+</segment>
+</net>
+<net name="2" class="0">
 <segment>
 <pinref part="U1" gate="A" pin="SCK"/>
-<pinref part="PAD3" gate="1" pin="P"/>
 <wire x1="45.72" y1="50.8" x2="38.1" y2="50.8" width="0.1524" layer="91"/>
-</segment>
-</net>
-<net name="N$4" class="0">
+<label x="40.64" y="50.8" size="1.778" layer="95"/>
+</segment>
+<segment>
+<pinref part="JP2" gate="A" pin="2"/>
+<wire x1="17.78" y1="45.72" x2="27.94" y2="45.72" width="0.1524" layer="91"/>
+<label x="22.86" y="45.72" size="1.778" layer="95"/>
+</segment>
+</net>
+<net name="3" class="0">
 <segment>
 <pinref part="U1" gate="A" pin="~RESET"/>
-<pinref part="PAD4" gate="1" pin="P"/>
 <wire x1="45.72" y1="48.26" x2="38.1" y2="48.26" width="0.1524" layer="91"/>
-<wire x1="38.1" y1="48.26" x2="38.1" y2="45.72" width="0.1524" layer="91"/>
-</segment>
-</net>
-<net name="N$5" class="0">
+<label x="40.64" y="48.26" size="1.778" layer="95"/>
+</segment>
+<segment>
+<pinref part="JP2" gate="A" pin="3"/>
+<wire x1="17.78" y1="48.26" x2="27.94" y2="48.26" width="0.1524" layer="91"/>
+<label x="22.86" y="48.26" size="1.778" layer="95"/>
+</segment>
+</net>
+<net name="4" class="0">
 <segment>
 <pinref part="U1" gate="A" pin="~CS"/>
-<wire x1="45.72" y1="45.72" x2="40.64" y2="45.72" width="0.1524" layer="91"/>
-<wire x1="40.64" y1="45.72" x2="40.64" y2="40.64" width="0.1524" layer="91"/>
-<pinref part="PAD5" gate="1" pin="P"/>
-<wire x1="40.64" y1="40.64" x2="38.1" y2="40.64" width="0.1524" layer="91"/>
-</segment>
-</net>
-<net name="N$6" class="0">
+<wire x1="45.72" y1="45.72" x2="38.1" y2="45.72" width="0.1524" layer="91"/>
+<label x="40.64" y="45.72" size="1.778" layer="95"/>
+</segment>
+<segment>
+<pinref part="JP2" gate="A" pin="4"/>
+<wire x1="17.78" y1="50.8" x2="27.94" y2="50.8" width="0.1524" layer="91"/>
+<label x="22.86" y="50.8" size="1.778" layer="95"/>
+</segment>
+</net>
+<net name="5" class="0">
 <segment>
 <pinref part="U1" gate="A" pin="~WP"/>
-<wire x1="45.72" y1="43.18" x2="43.18" y2="43.18" width="0.1524" layer="91"/>
-<wire x1="43.18" y1="43.18" x2="43.18" y2="35.56" width="0.1524" layer="91"/>
-<pinref part="PAD6" gate="1" pin="P"/>
-<wire x1="43.18" y1="35.56" x2="38.1" y2="35.56" width="0.1524" layer="91"/>
-</segment>
-</net>
-<net name="N$7" class="0">
+<wire x1="45.72" y1="43.18" x2="38.1" y2="43.18" width="0.1524" layer="91"/>
+<label x="40.64" y="43.18" size="1.778" layer="95"/>
+</segment>
+<segment>
+<pinref part="JP1" gate="A" pin="1"/>
+<wire x1="104.14" y1="58.42" x2="93.98" y2="58.42" width="0.1524" layer="91"/>
+<label x="93.98" y="58.42" size="1.778" layer="95"/>
+</segment>
+</net>
+<net name="7" class="0">
 <segment>
 <pinref part="U1" gate="A" pin="GND"/>
-<wire x1="45.72" y1="38.1" x2="45.72" y2="30.48" width="0.1524" layer="91"/>
-<pinref part="PAD7" gate="1" pin="P"/>
-<wire x1="45.72" y1="30.48" x2="38.1" y2="30.48" width="0.1524" layer="91"/>
-</segment>
-</net>
-<net name="N$8" class="0">
+<wire x1="45.72" y1="38.1" x2="38.1" y2="38.1" width="0.1524" layer="91"/>
+<label x="40.64" y="38.1" size="1.778" layer="95"/>
+</segment>
+<segment>
+<pinref part="JP1" gate="A" pin="3"/>
+<wire x1="104.14" y1="53.34" x2="93.98" y2="53.34" width="0.1524" layer="91"/>
+<label x="93.98" y="53.34" size="1.778" layer="95"/>
+</segment>
+</net>
+<net name="8" class="0">
 <segment>
 <pinref part="U1" gate="A" pin="SO"/>
-<pinref part="PAD8" gate="1" pin="P"/>
 <wire x1="81.28" y1="58.42" x2="88.9" y2="58.42" width="0.1524" layer="91"/>
+<label x="83.82" y="58.42" size="1.778" layer="95"/>
+</segment>
+<segment>
+<pinref part="JP1" gate="A" pin="4"/>
+<wire x1="104.14" y1="50.8" x2="93.98" y2="50.8" width="0.1524" layer="91"/>
+<label x="93.98" y="50.8" size="1.778" layer="95"/>
 </segment>
 </net>
@@
 </schematic>
 </drawing>
+<compatibility>
+<note version="8.2" severity="warning">
+Since Version 8.2, EAGLE supports online libraries. The ids
+of those online libraries will not be understood (or retained)
+with this version.
+</note>
+<note version="8.3" severity="warning">
+Since Version 8.3, EAGLE supports URNs for individual library
+assets (packages, symbols, and devices). The URNs of those assets
+will not be understood (or retained) with this version.
+</note>
+<note version="8.3" severity="warning">
+Since Version 8.3, EAGLE supports the association of 3D packages
+with devices in libraries, schematics, and board files. Those 3D
+packages will not be understood (or retained) with this version.
+</note>
+</compatibility>
 </eagle>
