File: Ethernet/main.brd (EAGLE design)
At the start: 87 x 47.5 mm, 35 parts, among them J1 J00-0045NL, P1 LAN8742A-CZ

Commit message: Ethernet PCB finalized
Parts:
- SV1: device con-lstb:MA05-2 -> con-lstb:MA06-2
- moved SV1 4.16 mm to (83.7, 67.5), turned to 270 degrees
- renumbered R9 to MDIO
Connections:
- net +3V3: now also SV1.11
- net GND: now also SV1.12
Routing:
- net GND: track 117.2 -> 138.3 mm, vias 3 -> 5
- net TXD1: track 24.4 -> 44.2 mm
- net NRST: track 20.7 -> 33.1 mm
- net N$1: track 19.1 -> 6.91 mm
- net +3V3: track 30.0 -> 40.7 mm
- net N$2: track 16.1 -> 7.04 mm
- net MDIO: track 22.4 -> 31.1 mm, vias 1 -> 2
- net TXD0: track 30.9 -> 39.7 mm, vias 2 -> 0
- net N$4: track 14.5 -> 7.17 mm
- net TXEN: track 23.7 -> 30.7 mm
- net MDC: track 19.5 -> 24.8 mm
- net N$5: track 11.0 -> 7.29 mm
- net RD_N: track 45.1 -> 44.6 mm
- net RD_P: track 48.5 -> 48.0 mm
- added copper zone on layer 1, net GND
- added copper zone on layer 16, net GND
Other:
- board size 87 x 47.5 mm -> 68.9 x 24.8 mm
