File: pdb_1.0.kicad_sch (KiCad schematic)
At the start: 64 parts, among them J1 Screw_Terminal_01x02, J10 Screw_Terminal_01x02, J2 Screw_Terminal_01x02, J3 Screw_Terminal_01x02, J7 Screw_Terminal_01x02, J8 Screw_Terminal_01x02, J9 Screw_Terminal_01x02, Q1 BSC340N08NS3G, Q2 BSC340N08NS3G, Q3 BSC340N08NS3G, Q4 BSC340N08NS3G, U1 LTC7891RUFDM-TRPBF, U2 LTC7891RUFDM-TRPBF

Commit message: chip layout, still need finalize a few peices and check for stock
Parts:
- removed C17: 0.1u, Capacitor_SMD:C_1206_3216Metric, symbol Device:C_Small
- added C26, C27, C28, C29: 0.1u, Capacitor_SMD:C_1206_3216Metric, symbol Device:C_Small
- added C30: 0.1u, Capacitor_SMD:CP_Elec_5x5.4, symbol Device:C_Small
- added R23, R24: 1M, Capacitor_SMD:C_0805_2012Metric, symbol Device:R_Small
- C14, C8: value 25n -> 50n
- C18: footprint Capacitor_SMD:C_1206_3216Metric -> Capacitor_SMD:CP_Elec_5x5.4
- C19: value 62p -> 65n
- C20: value 5.6p -> 9.9n
- C21: value 1800p -> 163n
- C22: value 27p -> 25n
- L1: value 47u -> 56u; footprint Inductor_SMD:L_Wuerth_HCF-2013 -> Inductor_SMD:L_Wuerth_HCI-2212
- L2: value 14u -> 33u; footprint Inductor_SMD:L_Wuerth_HCF-2013 -> Inductor_SMD:L_Wuerth_HCI-1890
- R1, R10: value 46.2k -> 374k
- R16: value 17m -> 15m
- R17, R8: value 60.4k -> 402k
- R18: value 7.87k -> 62k
- R19: value 442k -> 674k
- R20: value 46.4k -> 268k
- R6: value 28m -> 22m
- R9: value 2.67k -> 22.6k
Connections:
- net +19V: now also C28.2, C29.2
- net +7V: now also C26.2, C27.2, C30.2
- net GND: now also U1.2 (MODE), U2.2 (MODE)
- net GNDPWR: now also C26.1, C27.1, C28.1, C29.1, C30.1
- net INTVcc: now also R24.2; no longer U1.18 (PGOOD), U1.2 (MODE)
- net INTVcc_7v: now also R23.2; no longer U2.18 (PGOOD), U2.2 (MODE)
- new net: R24.1, U1.18 (PGOOD)
- new net: R23.1, U2.18 (PGOOD)
Other:
- note added: "24 - 15V Buck Converter"
- note added: "24 - 6V Buck Converter"
- note added: "MCU rail current draw: 240mA x 5 + 75mA x 4 + 5mA"
- note removed: "24 - 19V Buck Converter"
- note removed: "24 - 7V Buck Converter"
- moved on the sheet: C10, C11, C12, C13, C14, C15, C16, C18, C21, C22, C23, C24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

Commit message: finshed all connection, need double checking datasheet and componenet availaibility on JLC
Connections:
- net GND is gone; now on net GNDA: C11.1, C13.1, C14.1, C6.1, C7.1, C8.1, R1.1, R10.1, U1.1 (PLLIN/SPREAD), U1.2 (MODE), U1.27 (DRVUV), U1.5 (TEST), U2.1 (PLLIN/SPREAD), U2.2 (MODE), U2.27 (DRVUV), U2.5 (TEST)
- net GNDPWR is gone; now on net GNDA: C1.2, C12.1, C18.1, C2.2, C23.1, C24.1, C25.1, C26.1, C27.1, C28.1, C29.1, C3.2, C30.1, C4.2, C5.2, J1.1 (Pin_1), J10.1 (Pin_1), J2.1 (Pin_1), J3.1 (Pin_1), J7.1 (Pin_1), J8.1 (Pin_1), J9.1 (Pin_1), Q2.1 (S), Q2.2 (S), Q2.3 (S), Q4.1 (S), Q4.2 (S), Q4.3 (S), U1.29 (GND), U2.29 (GND)
