File: michael-main.kicad_sch (KiCad schematic)
At the start: 6 parts, among them J1 CAN, U1 STM32F446RETx, U2 MCP2551-I-SN

Commit message: initial board sch
Parts:
- added C10, C11, C13, C15, C16, C7, C8, C9: 0.1uF, Capacitor_SMD:C_0603_1608Metric, symbol Device:C_Small
- added C12, C6: 10uF, Capacitor_SMD:C_0603_1608Metric, symbol Device:C_Small
- added C14: 1uF, Capacitor_SMD:C_0603_1608Metric, symbol Device:C_Small
- added C2: C_Small, symbol Device:C_Small
- added C3, C4: 20pF, symbol Device:C_Small
- added C5: 4.7uF, Capacitor_SMD:C_0603_1608Metric, symbol Device:C_Small
- added D1: LED, LED_SMD:LED_0603_1608Metric, symbol Device:LED
- added FB1: 30R/1.8A, Inductor_SMD:L_0603_1608Metric, symbol Device:FerriteBead_Small
- added J2: USB_B_Mini, symbol Connector:USB_B_Mini
- added J3: Conn_01x05_Pin, symbol Connector:Conn_01x05_Pin
- added J4: PPTC041LGBN-RC, CONN_PPTC041LGBN-RC_SUL, symbol pptc041LGBN-RC:PPTC041LGBN-RC
- added J5: Conn_01x03_Pin, symbol Connector:Conn_01x03_Pin
- added R3: R_Small, symbol Device:R_Small
- added R4: 1k, Resistor_SMD:R_0603_1608Metric, symbol Device:R_Small
- added R5, R6: 4k, Resistor_SMD:R_0603_1608Metric, symbol Device:R_Small
- added R7: 10k, Resistor_SMD:R_0603_1608Metric, symbol Device:R_Small
- added U2, U3, U4, U5: STM32F446RETx, Package_QFP:LQFP-64_10x10mm_P0.5mm, symbol MCU_ST_STM32F4:STM32F446RETx
- added U7: USBLC6-4SC6, Package_TO_SOT_SMD:SOT-23-6, symbol Power_Protection:USBLC6-4SC6
- added U8: BMI088, BMI088:PQFN50P450X300X100-16N, symbol bmi088:BMI088
- added Y1: 8Mhz, symbol Device:Crystal
- added Y2, Y3, Y4: Crystal, symbol Device:Crystal
- renumbered U2 to U6
Connections:
- net GND: now also U1.12 (VSSA), U1.18 (VSS), U1.31 (VSS), U1.47 (VSS), U1.63 (VSS), C10.2, C11.2, C12.2, C13.2, C14.2, C15.1, C16.2, C3.2, C4.2, C5.2, C6.2, C7.2, C8.2, C9.2, D1.1 (K), J2.5 (GND), J3.3 (Pin_3), J4.1, J5.3 (Pin_3), R6.1, U7.2 (GND), U8.10 (SDO2), U8.15 (SDO1), U8.2 (NC), U8.4 (GNDA), U8.6 (GNDIO)
- net +3.3V: now reaches U1.1 (VBAT)
- net +3.3V: now also U1.19 (VDD), U1.32 (VDD), U1.48 (VDD), U1.64 (VDD), C10.1, C11.1, C14.1, C16.1, C6.1, C7.1, C8.1, C9.1, FB1.2, J3.1 (Pin_1), J4.2, J5.1 (Pin_1), R5.2, U8.11 (VDDIO), U8.3 (VDD), U8.7 (PS)
- net +3.3VA: now reaches U1.13 (VDDA)
- net +3.3VA: now also C12.1, C13.1, FB1.1
- net V_shunt_read: now reaches U1.23 (PA7)
- net Screen_SCL: now reaches U1.29 (PB10)
- net Screen_SCL: now also J4.3
- net at U1.30 (VCAP_1): now also C5.1
- net USB_D-: now reaches U1.44 (PA11)
- net USB_D-: now also U7.3 (I/O2)
- net USB_D+: now reaches U1.45 (PA12)
- net USB_D+: now also U7.1 (I/O1)
- net TMS1: now reaches U1.46 (PA13)
- net TMS1: now also J3.4 (Pin_4)
- net TCK1: now reaches U1.49 (PA14)
- net TCK1: now also J3.2 (Pin_2)
- net at U1.5 (PH0): now also C3.1, Y1.1
- net at U1.50 (PA15): now also R4.1
- net Screen_SDA: now reaches U1.55 (PB3)
- net Screen_SDA: now also J4.4
- net SCK_SCL: now reaches U1.58 (PB6)
- net SCK_SCL: now also R5.1, U8.8 (SCL/SCK)
- net SDI_SDA: now reaches U1.59 (PB7)
- net SDI_SDA: now also R6.2, U8.9 (SDA/SDI)
- net at U1.6 (PH1): now also C4.1, Y1.2
- net at U1.60 (BOOT0): now also R7.2
- net NRST1: now reaches U1.7 (NRST)
- net NRST1: now also C15.2, J3.5 (Pin_5)
- net INT1: now reaches U1.8 (PC0)
- net INT1: now also U8.16 (INT1)
- net INT3: now reaches U1.9 (PC1)
- net INT3: now also U8.12 (INT3)
- new net: U5.18 (VSS), U5.31 (VSS), U5.47 (VSS), U5.63 (VSS)
- new net: D1.2 (A), R4.2
- new net: J5.2 (Pin_2), R7.1
- new net: U2.18 (VSS), U2.31 (VSS), U2.47 (VSS), U2.63 (VSS)
- new net: U3.18 (VSS), U3.31 (VSS), U3.47 (VSS), U3.63 (VSS)
- new net: U4.18 (VSS), U4.31 (VSS), U4.47 (VSS), U4.63 (VSS)
- new net USB_CONN_D+: J2.3 (D+), U7.6 (I/O4)
- new net USB_CONN_D-: J2.2 (D-), U7.4 (I/O3)
- new net VBUS: J2.1 (VBUS), U7.5 (VBUS)
Other:
- moved on the sheet: C1, J1, R1, R2, U1, U6

Commit message: updated schematic and pcb; now need to add spi pins
Parts:
- added C17, C18, C19: 10uF, Capacitor_SMD:C_0805_2012Metric, symbol Device:C_Small
- added C20, C25, C28, C33, C36, C38, C44, C49: 10uF, Capacitor_SMD:C_0603_1608Metric, symbol Device:C_Small
- added C21, C22, C23, C24, C26, C29, C30, C31, C32, C34, C37, C39, C40, C41, C42, C43, C45, C47, C48, C50, C63, C64, C65: 0.1uF, Capacitor_SMD:C_0603_1608Metric, symbol Device:C_Small
- added C27, C35, C46, C51: 1uF, Capacitor_SMD:C_0603_1608Metric, symbol Device:C_Small
- added C52, C53, C54: C_Small, Capacitor_SMD:C_0805_2012Metric, symbol Device:C_Small
- added C55, C56, C57, C58, C59, C60, C61, C62: 20pF, Capacitor_SMD:C_0603_1608Metric, symbol Device:C_Small
- added FB2, FB3, FB4, FB5: 30R/1.8A, Inductor_SMD:L_0603_1608Metric, symbol Device:FerriteBead_Small
- added J10, J12, J8: CAN, Connector_JST:JST_GH_BM02B-GHS-TBT_1x02-1MP_P1.25mm_Vertical, symbol Connector:Conn_01x02_Pin
- added J11, J6, J7, J9: Conn_01x05_Pin, Connector_PinHeader_2.54mm:PinHeader_1x05_P2.54mm_Vertical, symbol Connector:Conn_01x05_Pin
- added J13, J14, J15, J16: Conn_01x03_Pin, Connector_PinHeader_2.54mm:PinHeader_1x03_P2.54mm_Vertical, symbol Connector:Conn_01x03_Pin
- added R10, R11, R12, R13, R8, R9: 60, Resistor_SMD:R_0805_2012Metric, symbol Device:R
- added R14, R15, R16: 10k, Resistor_SMD:R_0603_1608Metric, symbol Device:R_Small
- added U10: LM1084-5.0, Package_TO_SOT_SMD:TO-263-3_TabPin4, symbol Regulator_Linear:LM1084-5.0
- added U11, U12, U13: MCP2551-I-SN, Package_SO:SOIC-8_3.9x4.9mm_P1.27mm, symbol Interface_CAN_LIN:MCP2551-I-SN
- added U9: LM1084-3.3, Package_TO_SOT_SMD:TO-263-3_TabPin4, symbol Regulator_Linear:LM1084-3.3
- added Y5: Crystal, Crystal:Crystal_HC49-U_Vertical, symbol Device:Crystal
- C1: footprint (none) -> Capacitor_SMD:C_0805_2012Metric
- C2: value C_Small -> 0.1uF; footprint (none) -> Capacitor_SMD:C_0603_1608Metric
- C3, C4: footprint (none) -> Capacitor_SMD:C_0603_1608Metric
- J1: footprint (none) -> Connector_JST:JST_GH_BM02B-GHS-TBT_1x02-1MP_P1.25mm_Vertical
- J2: footprint (none) -> usb:USB_MINI
- J3: footprint (none) -> Connector_PinHeader_2.54mm:PinHeader_1x05_P2.54mm_Vertical
- J5: footprint (none) -> Connector_PinHeader_2.54mm:PinHeader_1x03_P2.54mm_Vertical
- R3: value R_Small -> 10k; footprint (none) -> Resistor_SMD:R_0603_1608Metric
- U8: footprint BMI088:PQFN50P450X300X100-16N -> bmi088:PQFN50P450X300X100-16N
- Y1, Y2, Y3, Y4: footprint (none) -> Crystal:Crystal_HC49-U_Vertical
Connections:
- net +3.3V: now also U2.1 (VBAT), U2.19 (VDD), U2.32 (VDD), U2.48 (VDD), U2.64 (VDD), U3.1 (VBAT), U3.19 (VDD), U3.32 (VDD), U3.48 (VDD), U3.64 (VDD), U4.1 (VBAT), U4.19 (VDD), U4.32 (VDD), U4.48 (VDD), U4.64 (VDD), U5.1 (VBAT), U5.19 (VDD), U5.32 (VDD), U5.48 (VDD), U5.64 (VDD), C19.1, C20.1, C21.1, C22.1, C23.1, C24.1, C27.1, C28.1, C29.1, C30.1, C31.1, C32.1, C35.1, C36.1, C37.1, C38.1, C39.1, C40.1, C41.1, C42.1, C43.1, C46.1, C47.1, C48.1, C51.1, FB2.2, FB3.2, FB4.2, FB5.2, J11.1 (Pin_1), J13.1 (Pin_1), J14.1 (Pin_1), J15.1 (Pin_1), J16.1 (Pin_1), J6.1 (Pin_1), J7.1 (Pin_1), J9.1 (Pin_1), U9.2 (VO)
- net +3.3VA: now also U2.13 (VDDA), U3.13 (VDDA), U4.13 (VDDA), U5.13 (VDDA), C25.1, C26.1, C33.1, C34.1, C44.1, C45.1, C49.1, C50.1, FB2.1, FB3.1, FB4.1, FB5.1
- net +5V: now also C18.1, U10.2 (VO), U11.3 (VDD), U12.3 (VDD), U13.3 (VDD), U9.3 (VI)
- net +6V: now also C17.1, U10.3 (VI)
- net GND: now also C2.1, U2.12 (VSSA), U2.18 (VSS), U2.31 (VSS), U2.47 (VSS), U2.63 (VSS), U3.12 (VSSA), U3.18 (VSS), U3.31 (VSS), U3.47 (VSS), U3.63 (VSS), U4.12 (VSSA), U4.18 (VSS), U4.31 (VSS), U4.47 (VSS), U4.63 (VSS), U5.12 (VSSA), U5.18 (VSS), U5.31 (VSS), U5.47 (VSS), U5.63 (VSS), C17.2, C18.2, C19.2, C20.2, C21.2, C22.2, C23.2, C24.2, C25.2, C26.2, C27.2, C28.2, C29.2, C30.2, C31.2, C32.2, C33.2, C34.2, C35.2, C36.2, C37.2, C38.2, C39.2, C40.2, C41.2, C42.2, C43.2, C44.2, C45.2, C46.2, C47.2, C48.2, C49.2, C50.2, C51.2, C55.2, C56.2, C57.2, C58.2, C59.2, C60.2, C61.2, C62.2, C63.1, C64.1, C65.1, J11.3 (Pin_3), J13.3 (Pin_3), J14.3 (Pin_3), J15.3 (Pin_3), J16.3 (Pin_3), J6.3 (Pin_3), J7.3 (Pin_3), J9.3 (Pin_3), U10.1 (GND), U11.2 (VSS), U11.8 (Rs), U12.2 (VSS), U12.8 (Rs), U13.2 (VSS), U13.8 (Rs), U9.1 (GND)
- net NRST1: now also J6.5 (Pin_5); no longer C15.2, J3.5 (Pin_5), U1.7 (NRST)
- net TCK1: now also J6.2 (Pin_2); no longer J3.2 (Pin_2), U1.49 (PA14)
- net TMS1: now also J6.4 (Pin_4); no longer J3.4 (Pin_4), U1.46 (PA13)
- net at Y2.1: now also U2.5 (PH0), C55.1
- net at Y2.2: now also U2.6 (PH1), C56.1
- net at U5.5 (PH0): now also C61.1, Y5.1
- net at U5.6 (PH1): now also C62.1, Y5.2
- net at U5.60 (BOOT0): now also R16.2
- net at U5.7 (NRST): now also C65.2
- net at C2.2: now also U2.7 (NRST)
- net at U2.60 (BOOT0): now also R3.2
- net at Y4.1: now also U4.5 (PH0), C59.1
- net at Y4.2: now also U4.6 (PH1), C60.1
- net at U3.5 (PH0): now also Y3.1, C57.1
- net at U3.6 (PH1): now also Y3.2, C58.1
- net at U3.60 (BOOT0): now also R14.2
- net at U3.7 (NRST): now also C63.2
- net at U4.60 (BOOT0): now also R15.2
- net at U4.7 (NRST): now also C64.2
- net at R3.1: now also J13.2 (Pin_2)
- net Vref_CAN renamed Vref1_CAN
- new net: C52.1, R8.2, R9.1
- new net: J16.2 (Pin_2), R16.1
- new net: C53.1, R10.2, R11.1
- new net: J10.1 (Pin_1), R11.2, U12.6 (CANL)
- new net: J10.2 (Pin_2), R10.1, U12.7 (CANH)
- new net: J14.2 (Pin_2), R14.1
- new net: J8.1 (Pin_1), R9.2, U11.6 (CANL)
- new net: J8.2 (Pin_2), R8.1, U11.7 (CANH)
- new net: J15.2 (Pin_2), R15.1
- new net: C54.1, R12.2, R13.1
- new net: J12.1 (Pin_1), R13.2, U13.6 (CANL)
- new net: J12.2 (Pin_2), R12.1, U13.7 (CANH)
- new net NRST: C15.2, J3.5 (Pin_5), U1.7 (NRST)
- new net NRST2: J7.5 (Pin_5)
- new net NRST3: J9.5 (Pin_5)
- new net NRST4: J11.5 (Pin_5)
- new net TCK: J3.2 (Pin_2), U1.49 (PA14)
- new net TCK2: J7.2 (Pin_2)
- new net TCK3: J9.2 (Pin_2)
- new net TCK4: J11.2 (Pin_2)
- new net TMS: J3.4 (Pin_4), U1.46 (PA13)
- new net TMS2: J7.4 (Pin_4)
- new net TMS3: J9.4 (Pin_4)
- new net TMS4: J11.4 (Pin_4)
- new net Vre4_CAN: U13.5 (Vref)
- new net Vref2_CAN: C52.2, U11.5 (Vref)
- new net Vref3_CAN: C53.2, U12.5 (Vref)
- new net Vref4_CAN: C54.2
Other:
- note added: "Master MCU"
- note added: "Power"
- note added: "Slave MCUs"
- moved on the sheet: C1, C16, J1, J2, R1, R2, U2, U3, U4, U5, U6, U7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

Commit message: updated estop circuit and buck converters for 16 and 6 volts, groups formed for pcb layout
Parts:
- added C37, C39, C40: 100u, Capacitor_SMD:C_Elec_10x10.2, symbol Device:C_Polarized_Small_US
- added C42: 1n, Capacitor_SMD:C_0805_2012Metric, symbol Device:C_Small
- added C51: 1u, Capacitor_SMD:C_0805_2012Metric, symbol Device:C_Small
- added C52, C53, C76, C77: 220u, Capacitor_SMD:C_Elec_6.3x7.7, symbol Device:C_Polarized_Small_US
- added C54, C58, C59, C63, C64, C66, C67, C74, C75: 0.1u, Capacitor_SMD:C_0805_2012Metric, symbol Device:C_Small
- added C55, C56: 10u, Capacitor_SMD:C_1206_3216Metric, symbol Device:C_Small
- added D2, D3: ss54, Diode_SMD:D_SMB, symbol Device:D_Schottky_Small
- added D4, D5: LED_Small, LED_SMD:LED_0805_2012Metric, symbol Device:LED_Small
- added H1, H2, H3, H4: MountingHole, MountingHole:MountingHole_3.2mm_M3, symbol Mechanical:MountingHole
- added J10, J11, J12, J13, J22: Conn_01x02_Pin, Connector_AMASS:AMASS_XT60PW-M_1x02_P7.20mm_Horizontal, symbol Connector:Conn_01x02_Pin
- added J14: Conn_01x02_Pin, Connector_AMASS:AMASS_XT90PW-M_1x02_P10.90mm_Horizontal, symbol Connector:Conn_01x02_Pin
- added J15: Conn_01x02_Pin, Connector_PinHeader_2.54mm:PinHeader_1x02_P2.54mm_Vertical, symbol Connector:Conn_01x02_Pin
- added L1: 6.8uH, Inductor_SMD:L_SXN_SMDRI124, symbol Device:L_Small
- added L2: 3uH, Inductor_SMD:L_Changjiang_FNR8040S, symbol Device:L_Small
- added Q1, Q2, Q3, Q4: BSC340N08NS3G, Package_TO_SOT_SMD:TDSON-8-1, symbol Transistor_FET:BSC340N08NS3G
- added R11: 10k, Resistor_SMD:R_0805_2012Metric, symbol Device:R_Small
- added R12: 1m, Resistor_SMD:R_2512_6332Metric, symbol Device:R_Small
- added R14, R15: 24k, Resistor_SMD:R_0805_2012Metric, symbol Device:R_Small
- added R16: 100k, Resistor_SMD:R_0805_2012Metric, symbol Device:R_Small
- added R17, R18: 0, Resistor_SMD:R_0805_2012Metric, symbol Device:R_Small
- added R19: 5, Resistor_SMD:R_0805_2012Metric, symbol Device:R_Small
- added R23: 380k, Resistor_SMD:R_0805_2012Metric, symbol Device:R_Small
- added R24, R26: 20k, Resistor_SMD:R_0805_2012Metric, symbol Device:R_Small
- added R25: 140k, Resistor_SMD:R_0805_2012Metric, symbol Device:R_Small
- added R27: 2.5k, Resistor_SMD:R_0805_2012Metric, symbol Device:R_Small
- added R28: 750, Resistor_SMD:R_0805_2012Metric, symbol Device:R_Small
- added U11, U12: LMR14050SDDAR, Package_SO:Texas_HSOP-8-1EP_3.9x4.9mm_P1.27mm_ThermalVias, symbol LMR14050SDDAR:LMR14050SDDAR
- added U8: LTC7000EMSE-1_TRPBF, ltc7000emse:SOP50P490X110-17N, symbol ltc7000emse:LTC7000EMSE-1_TRPBF
- renumbered C20 to C1, C23 to C10, C56 to C11, C4 to C12, C9 to C13, C15 to C14, C5 to C15, C24 to C16, C10 to C17, C11 to C18, C25 to C19, C6 to C2, C12 to C20, C26 to C21, C1 to C22, C13 to C23, C27 to C24, C14 to C25, C28 to C26, C29 to C27, C63 to C28, C57 to C29, C21 to C3, C58 to C31, C31 to C32, C32 to C33, C16 to C34, C33 to C35, C34 to C36, C35 to C38, C7 to C4, C52 to C41, C38 to C43, C39 to C44, C40 to C45, C64 to C46, C59 to C47, C41 to C48, C60 to C49, C2 to C5, C42 to C50, C44 to C57, C22 to C6, C45 to C60, C46 to C61, C53 to C62, C36 to C65, C37 to C68, C43 to C69, C55 to C7, C65 to C70, C61 to C71, C47 to C72, C62 to C73, C48 to C78, C17 to C79, C49 to C80, C50 to C81, C18 to C82, C51 to C83, C19 to C84, C54 to C85, C3 to C9, FB2 to FB1, FB1 to FB2, J13 to J1, J8 to J16, J15 to J17, J9 to J18, J16 to J19, J4 to J2, J10 to J20, J11 to J21, J12 to J24, J5 to J3, J6 to J4, J3 to J5, J1 to J6, J14 to J7, J2 to J8, J7 to J9, R3 to R1, R9 to R10, R15 to R13, R7 to R2, R10 to R20, R11 to R21, R16 to R22, R12 to R29, R1 to R3, R13 to R30, R2 to R4, R4 to R5, R5 to R6, R6 to R7, R14 to R8, R8 to R9, U2 to U1, U12 to U10, U5 to U13, U10 to U14, U13 to U15, U9 to U16, U6 to U2, U1 to U3, U8 to U4, U7 to U5, U3 to U6, U11 to U7, U4 to U9, Y2 to Y1, Y1 to Y2
Connections:
- net +3.3V: now also R11.2
- net +6V: now also C74.1, C77.1, L2.2, R25.1, R28.1
- net GND: now also C37.2, C39.2, C40.2, C42.2, C51.1, C52.2, C53.2, C55.2, C56.2, C58.2, C59.2, C63.2, C64.2, C74.2, C75.2, C76.2, C77.2, D2.2 (A), D3.2 (A), D4.1 (K), D5.1 (K), J10.1 (Pin_1), J11.1 (Pin_1), J12.1 (Pin_1), J13.1 (Pin_1), J14.1 (Pin_1), J15.2 (Pin_2), J22.1 (Pin_1), R14.2, R15.2, R24.2, R26.2, U11.10 (EXP__1), U11.11 (EXP__2), U11.12 (EXP__3), U11.13 (EXP__4), U11.14 (EXP__5), U11.15 (EXP__6), U11.16 (EXP__7), U11.17 (EXP__8), U11.7 (GND), U11.9 (EXP), U12.10 (EXP__1), U12.11 (EXP__2), U12.12 (EXP__3), U12.13 (EXP__4), U12.14 (EXP__5), U12.15 (EXP__6), U12.16 (EXP__7), U12.17 (EXP__8), U12.7 (GND), U12.9 (EXP), U8.17 (GND)
- new net: C66.1, U12.1 (BOOT)
- new net: R15.1, U12.4 (RT/SYNC)
- new net: R25.2, R26.1, U12.5 (FB)
- new net: C63.1, U12.6 (SS)
- new net: C66.2, D3.1 (K), L2.1, U12.8 (SW)
- new net: R12.1, U8.14 (SNS-)
- new net: D5.2 (A), R28.2
- new net: Q1.4 (G), Q2.4 (G), Q3.4 (G), Q4.4 (G), R19.1
- new net: R17.2, R18.2, R19.2
- new net: C51.2, R16.1, U8.3 (VCC)
- new net: R16.2, U8.6 (~{FAULT})
- new net: C67.1, U11.1 (BOOT)
- new net: C67.2, D2.1 (K), L1.1, U11.8 (SW)
- new net: D4.2 (A), R27.2
- new net: J15.1 (Pin_1), R11.1, U8.8 (INP)
- new net: C54.2, Q1.1 (S), Q1.2 (S), Q1.3 (S), Q2.1 (S), Q2.2 (S), Q2.3 (S), Q3.1 (S), Q3.2 (S), Q3.3 (S), Q4.1 (S), Q4.2 (S), Q4.3 (S), U8.11 (TS)
- new net: Q1.5 (D), Q2.5 (D), Q3.5 (D), Q4.5 (D)
- new net: C42.1, U8.7 (TIMER)
- new net: R23.2, R24.1, U11.5 (FB)
- new net: R17.1, U8.10 (TGUP)
- new net: C54.1, U8.12 (BST)
- new net: R18.1, U8.9 (TGDN)
- new net: R14.1, U11.4 (RT/SYNC)
- new net: C64.1, U11.6 (SS)
- new net +15V: C75.1, C76.1, J22.2 (Pin_2), L1.2, R23.1, R27.1
- new net +24V: C37.1, C39.1, C40.1, C52.1, C53.1, C55.1, C56.1, C58.1, C59.1, J10.2 (Pin_2), J11.2 (Pin_2), J12.2 (Pin_2), J13.2 (Pin_2), J14.2 (Pin_2), U11.2 (VIN), U12.2 (VIN)
- new net +BATT: R12.2, U8.1 (VIN), U8.16 (SNS+)
Other:
- moved on the sheet: C12, C13, C14, C15, C17, C18, C2, C20, C23, C25, C34, C4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

Commit message: finished componetnes placement, now need to add traces and pours
Parts:
- removed C34: 0.1uF, Capacitor_SMD:C_0603_1608Metric, symbol Device:C_Small
- removed C37, C39, C40: 100u, Capacitor_SMD:C_Elec_10x10.2, symbol Device:C_Polarized_Small_US
- removed J10, J11, J12, J13: Conn_01x02_Pin, Connector_AMASS:AMASS_XT60PW-M_1x02_P7.20mm_Horizontal, symbol Connector:Conn_01x02_Pin
- removed J16, J20, J24, J6: CAN, Connector_JST:JST_GH_BM02B-GHS-TBT_1x02-1MP_P1.25mm_Vertical, symbol Connector:Conn_01x02_Pin
- removed U4: BMI088, bmi088:PQFN50P450X300X100-16N, symbol bmi088:BMI088
- added J23: Conn_01x09_Socket, symbol Connector:Conn_01x09_Socket
- added J25: Conn_01x09_Socket, Connector_PinSocket_1.27mm:PinSocket_1x09_P1.27mm_Vertical, symbol Connector:Conn_01x09_Socket
- added J26: Conn_01x07_Socket, symbol Connector:Conn_01x07_Socket
- added J27: Conn_01x07_Socket, Connector_PinSocket_1.27mm:PinSocket_1x07_P1.27mm_Vertical, symbol Connector:Conn_01x07_Socket
- added J28, J29, J30, J31: XT30PW_2_2_-M.G.B, xt302+2:AMASS_XT30PW_2_2_-M.G.B, symbol xt302+2:XT30PW_2_2_-M.G.B
Connections:
- net Vre4_CAN is gone; now on net Vref4_CAN: U15.5 (Vref)
- net +24V: now also C54.2, Q1.1 (S), Q1.2 (S), Q1.3 (S), Q2.1 (S), Q2.2 (S), Q2.3 (S), Q3.1 (S), Q3.2 (S), Q3.3 (S), Q4.1 (S), Q4.2 (S), Q4.3 (S), U8.11 (TS), J28.P, J29.P, J30.P, J31.P; no longer C52.1, C53.1, C55.1, C56.1, C58.1, C59.1, J14.2 (Pin_2), U11.2 (VIN), U12.2 (VIN)
- net +3.3V: now also J25.6 (Pin_6), J27.1 (Pin_1), J27.2 (Pin_2)
- net +BATT: now also C52.1, C53.1, C55.1, C56.1, C58.1, C59.1, J14.2 (Pin_2), U11.2 (VIN), U12.2 (VIN)
- net GND: now also J25.3 (Pin_3), J27.3 (Pin_3), J28.N, J29.N, J30.N, J31.N
- net INT1: now also J27.6 (Pin_6)
- net NRST1: now also C5.2, U1.7 (NRST)
- net NRST2: now also C28.2, U6.7 (NRST)
- net NRST3: now also C46.2, U9.7 (NRST)
- net NRST4: now also C70.2, U13.7 (NRST)
- net SCK_SCL: now also J25.2 (Pin_2)
- net SDI_SDA: now also J25.4 (Pin_4)
- net TCK1: now also U1.49 (PA14)
- net TCK2: now also U6.49 (PA14)
- net TCK3: now also U9.49 (PA14)
- net TCK4: now also U13.49 (PA14)
- net TMS1: now also U1.46 (PA13)
- net TMS2: now also U6.46 (PA13)
- net TMS3: now also U9.46 (PA13)
- net TMS4: now also U13.46 (PA13)
- net sen-: now reaches R12.1, U8.14 (SNS-)
- net sen-: now also Q1.5 (D), Q2.5 (D), Q3.5 (D), Q4.5 (D)
- net INT3 renamed INT2
- net INT2: now also J27.7 (Pin_7)
Other:
- moved on the sheet: J14

Commit message: finished all traces for pcb, including power and mcu sections. 1. need to look into 15V jetson power ripple (ldo) 2. pgnd and agnd seperation, star connection, 0 ohm connnection, or solder paste connection at front layer. 3. isolate osc sources 4. remove non-conducting layers for motor power lines front and back
Parts:
- removed C74: 0.1u, Capacitor_SMD:C_0805_2012Metric, symbol Device:C_Small
- removed D4, D5: LED_Small, LED_SMD:LED_0805_2012Metric, symbol Device:LED_Small
- removed J23: Conn_01x09_Socket, symbol Connector:Conn_01x09_Socket
- removed J26: Conn_01x07_Socket, symbol Connector:Conn_01x07_Socket
- removed R27: 2.5k, Resistor_SMD:R_0805_2012Metric, symbol Device:R_Small
- removed R28: 750, Resistor_SMD:R_0805_2012Metric, symbol Device:R_Small
- removed U10, U15, U2, U7: MCP2551-I-SN, Package_SO:SOIC-8_3.9x4.9mm_P1.27mm, symbol Interface_CAN_LIN:MCP2551-I-SN
- added C34, C37, C39, C40: 0.1uF, Capacitor_SMD:C_0603_1608Metric, symbol Device:C_Small
- added D4: DFLS1150, Diode_SMD:D_PowerDI-123, symbol Device:D_Schottky_Small
- added D6, D7, D8, D9: NUP2105L, Package_TO_SOT_SMD:SOT-23, symbol Power_Protection:NUP2105L
- added R31, R32, R33: 5, Resistor_SMD:R_0805_2012Metric, symbol Device:R_Small
- added U17, U18, U2, U4: SN65HVD230, Package_SO:SOIC-8_3.9x4.9mm_P1.27mm, symbol Interface_CAN_LIN:SN65HVD230
- C22, C41, C62, C85: value C_Small -> 47n; footprint Capacitor_SMD:C_0805_2012Metric -> Capacitor_SMD:C_0603_1608Metric
- C79: footprint Capacitor_SMD:C_0805_2012Metric -> Capacitor_SMD:C_1206_3216Metric
- H1, H2, H3, H4: footprint MountingHole:MountingHole_3.2mm_M3 -> MountingHole:MountingHole_2.2mm_M2
Connections:
- net V_shunt_read is gone; now on net SPI_MOSI: U3.23 (PA7)
- net +24V: now also D4.1 (K)
- net +3.3V: now also C34.1, C37.1, C39.1, C40.1, U17.3 (VCC), U18.3 (VCC), U2.3 (VCC), U4.3 (VCC)
- net GND: now also C22.2, C41.2, C62.2, C85.2, C34.2, C37.2, C39.2, C40.2, D4.2 (A), D6.3 (A), D7.3 (A), D8.3 (A), D9.3 (A), U17.2 (GND), U17.8 (Rs), U18.2 (GND), U18.8 (Rs), U2.2 (GND), U2.8 (Rs), U4.2 (GND), U4.8 (Rs)
- net Vref1_CAN: now also C22.1, R3.2, R4.1, U4.5 (Vref); no longer C22.2
- net Vref2_CAN: now also C41.1, R10.1, R9.2, U2.5 (Vref); no longer C41.2
- net Vref3_CAN: now also C62.1, R20.2, R21.1, U17.5 (Vref); no longer C62.2
- net Vref4_CAN: now also C85.1, R29.2, R30.1, U18.5 (Vref); no longer C85.2
- net CS3: now reaches U13.20 (PA4)
- net CS3: now also U3.37 (PC6)
- net SPI_SCK: now reaches U13.21 (PA5)
- net SPI_SCK: now also U1.21 (PA5), U3.21 (PA5), U6.21 (PA5), U9.21 (PA5)
- net SPI_MISO: now reaches U13.22 (PA6)
- net SPI_MISO: now also U1.22 (PA6), U3.22 (PA6), U6.22 (PA6), U9.22 (PA6)
- net SPI_MOSI: now reaches U13.23 (PA7)
- net SPI_MOSI: now also U1.23 (PA7), U6.23 (PA7), U9.23 (PA7)
- net CAN4_RX: now reaches U13.44 (PA11)
- net CAN4_RX: now also U18.4 (R)
- net CAN4_TX: now reaches U13.45 (PA12)
- net CAN4_TX: now also U18.1 (D)
- net at R17.2, R18.2, R19.2: now also R31.2, R32.2, R33.2
- net CANL1: now reaches R4.2
- net CANL1: now also J29.S2, D6.1 (K), U4.6 (CANL)
- net CANH1: now reaches R3.1
- net CANH1: now also J29.S1, D6.2 (K), U4.7 (CANH)
- net CANL3: now reaches R21.2
- net CANL3: now also J31.S2, D8.1 (K), U17.6 (CANL)
- net CANH3: now reaches R20.1
- net CANH3: now also J31.S1, D8.2 (K), U17.7 (CANH)
- net CANL4: now reaches R30.2
- net CANL4: now also J28.S2, D9.1 (K), U18.6 (CANL)
- net CANH2: now reaches R9.1
- net CANH2: now also J30.S1, D7.2 (K), U2.7 (CANH)
- net CANL2: now reaches J30.S2
- net CANL2: now also R10.2, D7.1 (K), U2.6 (CANL)
- net CANH4: now reaches R29.1
- net CANH4: now also J28.S1, D9.2 (K), U18.7 (CANH)
- net CS2: now reaches U1.20 (PA4)
- net CS2: now also U3.38 (PC7)
- net CAN1_RX: now reaches U1.44 (PA11)
- net CAN1_RX: now also U4.4 (R)
- net CAN1_TX: now reaches U1.45 (PA12)
- net CAN1_TX: now also U4.1 (D)
- net CS0: now reaches U6.20 (PA4)
- net CS0: now also U3.40 (PC9)
- net CAN2_RX: now reaches U6.44 (PA11)
- net CAN2_RX: now also U2.4 (R)
- net CAN2_TX: now reaches U6.45 (PA12)
- net CAN2_TX: now also U2.1 (D)
- net CS1: now reaches U9.20 (PA4)
- net CS1: now also U3.39 (PC8)
- net CAN3_RX: now reaches U9.44 (PA11)
- net CAN3_RX: now also U17.4 (R)
- net CAN3_TX: now reaches U9.45 (PA12)
- net CAN3_TX: now also U17.1 (D)
- net SPI_NSS: now reaches U3.20 (PA4)
- removed net +3.3VA: C19.1, C20.1, C21.1, C23.1, C35.1, C36.1, C57.1, C60.1, C80.1, C81.1, FB1.1, FB2.1, FB3.1, FB4.1, FB5.1, U1.13 (VDDA), U13.13 (VDDA), U3.13 (VDDA), U6.13 (VDDA), U9.13 (VDDA)
- new net +3.3V5: C80.1, C81.1, FB5.1, U13.13 (VDDA)
- new net +3.3VA1: C20.1, C23.1, FB2.1, U3.13 (VDDA)
- new net +3.3VA2: C19.1, C21.1, FB1.1, U1.13 (VDDA)
- new net +3.3VA3: C35.1, C36.1, FB3.1, U6.13 (VDDA)
- new net +3.3VA4: C57.1, C60.1, FB4.1, U9.13 (VDDA)
- new net G1: Q1.4 (G), R33.1
- new net G2: Q2.4 (G), R32.1
- new net G3: Q3.4 (G), R31.1
- new net G4: Q4.4 (G), R19.1
Other:
- moved on the sheet: C22, C41, C51, C54, C62, C85, R16, R17, R18, R19, R29, R30

Commit message: finished solder mask removal, switched to a smaller crystal, finished osc signal isolation
Parts:
- Y1, Y2, Y3, Y4, Y5: footprint Crystal:Crystal_HC49-U_Vertical -> Crystal:Crystal_SMD_5032-4Pin_5.0x3.2mm
Changed lines of the file:
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@@
 			)
 		)
-		(property "Footprint" "Crystal:Crystal_HC49-U_Vertical"
+		(property "Footprint" "Crystal:Crystal_SMD_5032-4Pin_5.0x3.2mm"
 			(at 55.88 77.47 0)
 			(effects
@@
 			)
 		)
-		(property "Footprint" "Crystal:Crystal_HC49-U_Vertical"
+		(property "Footprint" "Crystal:Crystal_SMD_5032-4Pin_5.0x3.2mm"
 			(at 53.34 247.65 0)
 			(effects
@@
 			)
 		)
-		(property "Footprint" "Crystal:Crystal_HC49-U_Vertical"
+		(property "Footprint" "Crystal:Crystal_SMD_5032-4Pin_5.0x3.2mm"
 			(at 486.41 248.92 0)
 			(effects
@@
 			)
 		)
-		(property "Footprint" "Crystal:Crystal_HC49-U_Vertical"
+		(property "Footprint" "Crystal:Crystal_SMD_5032-4Pin_5.0x3.2mm"
 			(at 179.07 247.65 0)
 			(effects
@@
 			)
 		)
-		(property "Footprint" "Crystal:Crystal_HC49-U_Vertical"
+		(property "Footprint" "Crystal:Crystal_SMD_5032-4Pin_5.0x3.2mm"
 			(at 334.01 247.65 0)
 			(effects

Commit message: edited master mcu section
Parts:
- removed J2: PPTC041LGBN-RC, CONN_PPTC041LGBN-RC_SUL, symbol pptc041LGBN-RC:PPTC041LGBN-RC
- R12: value 1m -> 0.5m
- U14, U16: footprint Package_TO_SOT_SMD:TO-263-3_TabPin4 -> Package_TO_SOT_SMD:TO-263-3_TabPin2
- Y1, Y2, Y3, Y4, Y5: footprint Crystal:Crystal_SMD_5032-4Pin_5.0x3.2mm -> Crystal:Crystal_HC49-U_Vertical
Connections:
- net Screen_SCL: no longer names the net of U3.29 (PB10)
- net Screen_SDA: no longer names the net of U3.55 (PB3)
