File: michael-main.kicad_sch (KiCad schematic)
At the start: 178 parts, among them J1 Conn_01x03_Pin, J14 Conn_01x02_Pin, J15 Conn_01x02_Pin, J17 Conn_01x03_Pin, J18 Conn_01x05_Pin, J19 Conn_01x03_Pin, J21 Conn_01x05_Pin, J22 Conn_01x02_Pin, J25 Conn_01x09_Socket, J27 Conn_01x07_Socket, J28 XT30PW_2_2_-M.G.B, J29 XT30PW_2_2_-M.G.B, J3 Conn_01x03_Pin, J30 XT30PW_2_2_-M.G.B, J31 XT30PW_2_2_-M.G.B, J4 Conn_01x05_Pin, J5 Conn_01x05_Pin, J7 Conn_01x03_Pin, J8 USB_B_Mini, J9 Conn_01x05_Pin, Q1 BSC340N08NS3G, Q2 BSC340N08NS3G, Q3 BSC340N08NS3G, Q4 BSC340N08NS3G, U1 STM32F446RETx, U11 LMR14050SDDAR, U12 LMR14050SDDAR, U13 STM32F446RETx, U14 LM1084-5.0, U16 LM1084-3.3, U17 SN65HVD230, U18 SN65HVD230, U2 SN65HVD230, U3 STM32F446RETx, U4 SN65HVD230, U5 USBLC6-4SC6, U6 STM32F446RETx, U8 LTC7000EMSE-1_TRPBF, U9 STM32F446RETx, Y1 Crystal, Y2 8Mhz, Y3 Crystal, Y4 Crystal, Y5 Crystal

Commit message: updated routing for shorter power trace
Parts:
- added J2: Conn_01x03_Pin, symbol Connector:Conn_01x03_Pin
- added R27, R28, R34, R35: 47k, Resistor_SMD:R_0402_1005Metric, symbol Device:R_Small
- added R36: 0, Resistor_SMD:R_0805_2012Metric, symbol Device:R_Small
- C1, C10, C13, C14, C16, C17, C18, C19, C2, C20, C21, C23, C24, C25, C26, C27, C28, C3, C30, C32, C33, C34, C35, C36, C37, C38, C39, C4, C40, C43, C44, C45, C46, C48, C5, C50, C57, C6, C60, C61, C65, C68, C69, C70, C72, C78, C8, C80, C81, C83: footprint Capacitor_SMD:C_0603_1608Metric -> Capacitor_SMD:C_0402_1005Metric
- J22: footprint Connector_AMASS:AMASS_XT60PW-M_1x02_P7.20mm_Horizontal -> Connector_AMASS:AMASS_XT60-M_1x02_P7.20mm_Vertical
- R1, R13, R2, R22, R8: footprint Resistor_SMD:R_0603_1608Metric -> Resistor_SMD:R_0402_1005Metric
- R11: footprint Resistor_SMD:R_0805_2012Metric -> Resistor_SMD:R_0402_1005Metric
- Y1, Y3, Y4, Y5: value Crystal -> 8Mhz
Connections:
- net +3.3V: now also J15.2 (Pin_2), R27.2, R28.2, R34.2, R35.2; no longer R11.2
- net CANH2: now also J31.S1; no longer J30.S1
- net CANH3: now also J30.S1; no longer J31.S1
- net CANL2: now also J31.S2; no longer J30.S2
- net CANL3: now also J30.S2; no longer J31.S2
- net CS0: now also R28.1
- net CS1: now also R34.1
- net CS2: now also R27.1
- net CS3: now also R35.1
- net GND: now also R11.2, R36.2; no longer C52.2, C53.2, C55.2, C56.2, C58.2, C59.2, C75.2, C76.2, C77.2, C79.2, C82.2, C84.2, D2.2 (A), D3.2 (A), J14.1 (Pin_1), J15.2 (Pin_2), J22.1 (Pin_1), J28.N, J29.N, J30.N, J31.N, R24.2, R26.2, U14.1 (GND), U16.1 (GND)
- net FB6: now reaches R25.2, R26.1, U12.5 (FB)
- net at C7.1, U1.5 (PH0): now also Y5.1; no longer Y1.1
- net at C11.1, U1.6 (PH1): now also Y5.2; no longer Y1.2
- net at C71.1, U13.5 (PH0): now also Y4.1; no longer Y5.1
- net at C73.1, U13.6 (PH1): now also Y4.2; no longer Y5.2
- net at C47.1, U9.5 (PH0): now also Y3.1; no longer Y4.1
- net at C49.1, U9.6 (PH1): now also Y3.2; no longer Y4.2
- net at C29.1, U6.5 (PH0): now also Y1.1; no longer Y3.1
- net at C31.1, U6.6 (PH1): now also Y1.2; no longer Y3.2
- net at J15.1 (Pin_1), R11.1: now also J2.1 (Pin_1); no longer U8.8 (INP)
- net FB15: now reaches R23.2, R24.1, U11.5 (FB)
- new net: J2.2 (Pin_2), U8.8 (INP)
- new net GNDPWR: C52.2, C53.2, C55.2, C56.2, C58.2, C59.2, C75.2, C76.2, C77.2, C79.2, C82.2, C84.2, D2.2 (A), D3.2 (A), J14.1 (Pin_1), J22.1 (Pin_1), J28.N, J29.N, J30.N, J31.N, R24.2, R26.2, R36.1, U14.1 (GND), U16.1 (GND)
- new net PWM: J2.3 (Pin_3)
Other:
- moved on the sheet: C52, C53, C55, C56, C58, C59, C70, C71, C73, C75, C76, C77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
