File: michael-main.kicad_sch (KiCad schematic)
At the start: 184 parts, among them J1 Conn_01x03_Pin, J14 Conn_01x02_Pin, J15 Conn_01x02_Pin, J17 Conn_01x03_Pin, J18 Conn_01x05_Pin, J19 Conn_01x03_Pin, J2 Conn_01x03_Pin, J21 Conn_01x05_Pin, J22 Conn_01x02_Pin, J25 Conn_01x09_Socket, J27 Conn_01x07_Socket, J28 XT30PW_2_2_-M.G.B, J29 XT30PW_2_2_-M.G.B, J3 Conn_01x03_Pin, J30 XT30PW_2_2_-M.G.B, J31 XT30PW_2_2_-M.G.B, J4 Conn_01x05_Pin, J5 Conn_01x05_Pin, J7 Conn_01x03_Pin, J8 USB_B_Mini, J9 Conn_01x05_Pin, Q1 BSC340N08NS3G, Q2 BSC340N08NS3G, Q3 BSC340N08NS3G, Q4 BSC340N08NS3G, U1 STM32F446RETx, U11 LMR14050SDDAR, U12 LMR14050SDDAR, U13 STM32F446RETx, U14 LM1084-5.0, U16 LM1084-3.3, U17 SN65HVD230, U18 SN65HVD230, U2 SN65HVD230, U3 STM32F446RETx, U4 SN65HVD230, U5 USBLC6-4SC6, U6 STM32F446RETx, U8 LTC7000EMSE-1_TRPBF, U9 STM32F446RETx, Y1 8Mhz, Y2 8Mhz, Y3 8Mhz, Y4 8Mhz, Y5 8Mhz

Commit message: competed
Parts:
- removed J15: Conn_01x02_Pin, Connector_PinHeader_2.54mm:PinHeader_1x02_P2.54mm_Vertical, symbol Connector:Conn_01x02_Pin
- removed J2: Conn_01x03_Pin, symbol Connector:Conn_01x03_Pin
- added C74: 0.1u, Capacitor_SMD:C_0805_2012Metric, symbol Device:C_Small
- added D10: 5.0SMDJ33A, Diode_SMD:D_SMC, symbol Diode:Z3SMCxxx
- added D5: LED, LED_SMD:LED_0603_1608Metric, symbol Device:LED
- added J6: Conn_01x03_Pin, Connector_JST:JST_XH_B3B-XH-A_1x03_P2.50mm_Vertical, symbol Connector:Conn_01x03_Pin
- added R37, R38: 22, Resistor_SMD:R_0603_1608Metric, symbol Device:R_Small
- added R39, R40: 0, Resistor_SMD:R_0402_1005Metric, symbol Device:R_Small
- added R41: 1k, Resistor_SMD:R_0603_1608Metric, symbol Device:R_Small
- C42, C51: footprint Capacitor_SMD:C_0805_2012Metric -> Capacitor_SMD:C_0603_1608Metric
- J14: footprint Connector_AMASS:AMASS_XT90PW-M_1x02_P10.90mm_Horizontal -> Connector_AMASS:AMASS_XT60PW-M_1x02_P7.20mm_Horizontal
- R12: footprint Resistor_SMD:R_2512_6332Metric -> wslp:RES_WSLP3921_.001OHM_VIS-L
- R16: footprint Resistor_SMD:R_0805_2012Metric -> Resistor_SMD:R_0603_1608Metric
- R17: value 0 -> 33k
- R18: value 0 -> 22
Connections:
- net +3.3V: now also J6.2 (Pin_2), J6.3 (Pin_3), R40.1, R41.2
- net GND: now also C74.1
- net GNDPWR: now also D10.2 (A), D5.1 (K)
- net SPI_MOSI: now also R38.2; no longer U3.23 (PA7)
- net SPI_SCK: now also R37.2; no longer U3.21 (PA5)
- net sen-: now also D10.1 (K)
- net at R17.2, R18.2, R19.2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: now also C74.2
- net PWR_CTL_IN: now reaches R11.1
- net PWR_CTL_IN: now also J6.1 (Pin_1), R39.1
- net at U8.8 (INP): now also R39.2, R40.2
- new net: R37.1, U3.21 (PA5)
- new net: D5.2 (A), R41.1
- new net: R38.1, U3.23 (PA7)
Other:
- moved on the sheet: R11

Commit message: updated vcap, reworked on power plane, added debug led and uart to 1 slave
Parts:
- removed H3: MountingHole, MountingHole:MountingHole_2.2mm_M2, symbol Mechanical:MountingHole
- removed R40: 0, Resistor_SMD:R_0402_1005Metric, symbol Device:R_Small
- removed U14: LM1084-5.0, Package_TO_SOT_SMD:TO-263-3_TabPin2, symbol Regulator_Linear:LM1084-5.0
- removed U5: USBLC6-4SC6, Package_TO_SOT_SMD:SOT-23-6, symbol Power_Protection:USBLC6-4SC6
- added C101, C90, C91, C92, C94, C95: 0.1u, Capacitor_SMD:C_0805_2012Metric, symbol Device:C_Small
- added C86, C87, C88, C89: 4.7uF, Capacitor_SMD:C_0402_1005Metric, symbol Device:C_Small
- added C93: 1n, Capacitor_SMD:C_0805_2012Metric, symbol Device:C_Small
- added C96: 10uF, Capacitor_SMD:C_0805_2012Metric, symbol Device:C_Small
- added C97: 10u, Capacitor_SMD:C_0805_2012Metric, symbol Device:C_Small
- added D11: 5.0SMDJ33A, Diode_SMD:D_SMC, symbol Diode:Z3SMCxxx
- added D13, D14, D15, D16, D17, D18, D19, D20, D21, D22, D27, D28, D29, D30: LED, LED_SMD:LED_0603_1608Metric, symbol Device:LED
- added J2: Conn_01x04_Pin, Connector_PinHeader_2.54mm:PinHeader_1x04_P2.54mm_Vertical, symbol Connector:Conn_01x04_Pin
- added R42: 22, Resistor_SMD:R_0603_1608Metric, symbol Device:R_Small
- added R43, R48, R49, R50: 0, Resistor_SMD:R_0603_1608Metric, symbol Device:R_Small
- added R44, R45: 11, Resistor_SMD:R_0603_1608Metric, symbol Device:R_Small
- added R46, R47, R51, R52, R53, R54, R55, R56, R57, R58, R63, R64, R65, R66: 1k, Resistor_SMD:R_0603_1608Metric, symbol Device:R_Small
- added U7: USBLC6-2SC6, Package_TO_SOT_SMD:SOT-23-6, symbol Power_Protection:USBLC6-2SC6
- C10, C13, C14, C16, C17, C18, C21, C23, C27, C28, C3, C30, C32, C33, C34, C36, C37, C39, C4, C40, C44, C45, C46, C48, C5, C50, C6, C60, C68, C69, C70, C72, C78, C8, C81: value 0.1uF -> 0.1u
- C55: footprint Capacitor_SMD:C_1206_3216Metric -> Capacitor_SMD:C_0805_2012Metric
- C56: value 10u -> 1n; footprint Capacitor_SMD:C_1206_3216Metric -> Capacitor_SMD:C_0805_2012Metric
- C82: value 10uF -> 0.1u
- R10, R20, R21, R29, R3, R30, R4, R9: value 60 -> 75; footprint Resistor_SMD:R_0805_2012Metric -> Resistor_SMD:R_0603_1608Metric
- R41: value 1k -> 8k
Connections:
- net +15V: now also C56.1, C90.1, C91.1, C93.1, C97.1
- net +24V: now also D10.1 (K)
- net +3.3V: now also C82.1, C101.1, C92.1, C96.1, J2.1 (Pin_1)
- net +6V: now also U16.3 (VI), C94.1, C95.1
- net +BATT: now also D11.1 (K); no longer C56.1
- net GND: now also C86.2, C87.2, C88.2, C89.2, D13.1 (K), D14.1 (K), D15.1 (K), D16.1 (K), D17.1 (K), D18.1 (K), D19.1 (K), D20.1 (K), D21.1 (K), D22.1 (K), D27.1 (K), D28.1 (K), D29.1 (K), D30.1 (K), J2.4 (Pin_4), R43.1, R48.1, R49.1, R50.1, U7.2 (GND); no longer U17.8 (Rs), U18.8 (Rs), U2.8 (Rs), U4.8 (Rs)
- net GNDPWR: now also C101.2, C90.2, C91.2, C92.2, C93.2, C94.2, C95.2, C96.2, C97.2, D11.2 (A)
- net SPI_MISO: now also R42.2; no longer U3.22 (PA6)
- net USB_CONN_D+: now also U7.6 (I/O1)
- net USB_CONN_D-: now also U7.4 (I/O2)
- net USB_D+: now also U7.1 (I/O1)
- net USB_D-: now also U7.3 (I/O2)
- net VBUS: now also U7.5 (VBUS)
- net sen-: no longer D10.1 (K)
- net at U13.30 (VCAP_1): now also C89.1
- net at U13.43 (PA10): now also R47.1
- net at U1.30 (VCAP_1): now also C86.1
- net at U1.33 (PB12): now also R66.1
- net at U1.34 (PB13): now also R65.1
- net at U1.35 (PB14): now also R64.1
- net at U1.36 (PB15): now also R63.1
- net at U6.30 (VCAP_1): now also C87.1
- net Slave_tx: now reaches U6.53 (PC12)
- net Slave_tx: now also R44.1
- net Slave_rx: now reaches U6.54 (PD2)
- net Slave_rx: now also R45.1
- net at U6.55 (PB3): now also R54.1
- net at U6.56 (PB4): now also R53.1
- net at U6.57 (PB5): now also R52.1
- net at U6.58 (PB6): now also R51.1
- net at U9.30 (VCAP_1): now also C88.1
- net at U9.36 (PB15): now also R46.1
- net at U3.33 (PB12): now also R58.1
- net at U3.34 (PB13): now also R57.1
- net at U3.35 (PB14): now also R56.1
- net at U3.36 (PB15): now also R55.1
- removed net +5V: C82.1, U16.3 (VI)
- new net: D16.2 (A), R52.2
- new net: R48.2, U2.8 (Rs)
- new net: D27.2 (A), R63.2
- new net: R49.2, U17.8 (Rs)
- new net: D18.2 (A), R54.2
- new net: J2.2 (Pin_2), R45.2
- new net: J2.3 (Pin_3), R44.2
- new net: D17.2 (A), R53.2
- new net: D30.2 (A), R66.2
- new net: R50.2, U18.8 (Rs)
- new net: D28.2 (A), R64.2
- new net: D19.2 (A), R55.2
- new net: D15.2 (A), R51.2
- new net: R43.2, U4.8 (Rs)
- new net: D13.2 (A), R46.2
- new net: D21.2 (A), R57.2
- new net: D14.2 (A), R47.2
- new net: D20.2 (A), R56.2
- new net: D22.2 (A), R58.2
- new net: R42.1, U3.22 (PA6)
- new net: D29.2 (A), R65.2
Other:
- moved on the sheet: C12, C13, C14, C17, C18, C2, C20, C23, C25, C4, C40, C75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

Commit message: schematic change
Parts:
- R6: value 4k -> 4.7k; footprint Resistor_SMD:R_0603_1608Metric -> Resistor_SMD:R_0402_1608Metric
- R7: value 4k -> 4.7k; footprint Resistor_SMD:R_0603_1608Metric -> Resistor_SMD:R_0402_1005Metric
Connections:
- net +3.3V: now also R7.1
- net GND: no longer R7.1
Other:
- moved on the sheet: R7
Changed lines of the file:
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@@
 	)
 	(junction
+		(at 149.86 111.76)
+		(diameter 0)
+		(color 0 0 0 0)
+	)
+	(junction
 		(at 373.38 116.84)
 		(diameter 0)
@@
 	(wire
 		(pts
-			(xy 114.3 124.46) (xy 142.24 124.46)
-		)
-		(stroke
-			(width 0)
-			(type default)
-		)
-	)
-	(wire
-		(pts
 			(xy 373.38 109.22) (xy 373.38 106.68)
 		)
@@
 	(wire
 		(pts
+			(xy 149.86 111.76) (xy 142.24 111.76)
+		)
+		(stroke
+			(width 0)
+			(type default)
+		)
+	)
+	(wire
+		(pts
 			(xy 384.81 248.92) (xy 389.89 248.92)
 		)
@@
 	(wire
 		(pts
-			(xy 142.24 129.54) (xy 142.24 130.81)
-		)
-		(stroke
-			(width 0)
-			(type default)
-		)
-	)
-	(wire
-		(pts
 			(xy 238.76 215.9) (xy 256.54 215.9)
 		)
@@
 	(wire
 		(pts
+			(xy 142.24 111.76) (xy 142.24 116.84)
+		)
+		(stroke
+			(width 0)
+			(type default)
+		)
+	)
+	(wire
+		(pts
 			(xy 457.2 212.09) (xy 467.36 212.09)
 		)
@@
 	(wire
 		(pts
+			(xy 149.86 111.76) (xy 149.86 116.84)
+		)
+		(stroke
+			(width 0)
+			(type default)
+		)
+	)
+	(wire
+		(pts
 			(xy 400.05 356.87) (xy 403.86 356.87)
 		)
@@
 	(wire
 		(pts
+			(xy 114.3 124.46) (xy 149.86 124.46)
+		)
+		(stroke
+			(width 0)
+			(type default)
+		)
+	)
+	(wire
+		(pts
 			(xy 443.23 163.83) (xy 454.66 163.83)
 		)
@@
 	(wire
 		(pts
-			(xy 142.24 114.3) (xy 142.24 116.84)
-		)
-		(stroke
-			(width 0)
-			(type default)
-		)
-	)
-	(wire
-		(pts
 			(xy 40.64 48.26) (xy 30.48 48.26)
 		)
@@
 	(wire
 		(pts
+			(xy 149.86 121.92) (xy 149.86 124.46)
+		)
+		(stroke
+			(width 0)
+			(type default)
+		)
+	)
+	(wire
+		(pts
 			(xy 264.16 312.42) (xy 264.16 313.69)
 		)
@@
 	)
 	(label "SCK_SCL"
-		(at 118.11 121.92 0)
+		(at 125.73 121.92 180)
 		(effects
 			(font
 				(size 1.27 1.27)
 			)
-			(justify left bottom)
+			(justify right bottom)
 		)
 	)
@@
 	)
 	(label "SDI_SDA"
-		(at 118.11 124.46 0)
+		(at 125.73 124.46 180)
 		(effects
 			(font
 				(size 1.27 1.27)
 			)
-			(justify left bottom)
+			(justify right bottom)
 		)
 	)
@@
 	)
 	(symbol
-		(lib_id "power:GND")
-		(at 142.24 130.81 0)
-		(unit 1)
-		(exclude_from_sim no)
-		(in_bom yes)
-		(on_board yes)
-		(dnp no)
-		(property "Reference" "#PWR033"
-			(at 142.24 137.16 0)
-			(effects
-				(font
-					(size 1.27 1.27)
-				)
-				(hide yes)
-			)
-		)
-		(property "Value" "GND"
-			(at 146.304 132.334 0)
-			(effects
-				(font
-					(size 1.27 1.27)
-				)
-			)
-		)
-		(property "Footprint" ""
-			(at 142.24 130.81 0)
-			(effects
-				(font
-					(size 1.27 1.27)
-				)
-				(hide yes)
-			)
-		)
-		(property "Datasheet" ""
-			(at 142.24 130.81 0)
-			(effects
-				(font
-					(size 1.27 1.27)
-				)
-				(hide yes)
-			)
-		)
-		(property "Description" "Power symbol creates a global label with name \"GND\" , ground"
-			(at 142.24 130.81 0)
-			(effects
-				(font
-					(size 1.27 1.27)
-				)
-				(hide yes)
-			)
-		)
-		(pin "1"
-		)
-		(instances
-			(project "michael-main"
-				(path "/034f55b6-c74d-4d81-b822-70258ab62f40"
-					(reference "#PWR033")
-					(unit 1)
-				)
-			)
-		)
-	)
-	(symbol
 		(lib_id "power:+3.3V")
 		(at 48.26 66.04 270)
@@
 			)
 		)
-		(property "Value" "4k"
+		(property "Value" "4.7k"
 			(at 144.78 120.6499 0)
 			(effects
@@
 			)
 		)
-		(property "Footprint" "Resistor_SMD:R_0603_1608Metric"
+		(property "Footprint" "Resistor_SMD:R_0402_1608Metric"
 			(at 142.24 119.38 0)
 			(effects
@@
 	(symbol
 		(lib_id "Device:R_Small")
-		(at 142.24 127 180)
+		(at 149.86 119.38 0)
 		(unit 1)
 		(exclude_from_sim no)
@@
 		(fields_autoplaced yes)
 		(property "Reference" "R7"
-			(at 144.78 125.7299 0)
+			(at 152.4 118.1099 0)
 			(effects
 				(font
 					(size 1.016 1.016)
 				)
-				(justify right)
+				(justify left)
 			)
 		)
-		(property "Value" "4k"
-			(at 144.78 128.2699 0)
+		(property "Value" "4.7k"
+			(at 152.4 120.6499 0)
 			(effects
 				(font
 					(size 1.27 1.27)
 				)
-				(justify right)
+				(justify left)
 			)
 		)
-		(property "Footprint" "Resistor_SMD:R_0603_1608Metric"
-			(at 142.24 127 0)
+		(property "Footprint" "Resistor_SMD:R_0402_1005Metric"
+			(at 149.86 119.38 0)
 			(effects
 				(font
@@
 		)
 		(property "Datasheet" "~"
-			(at 142.24 127 0)
+			(at 149.86 119.38 0)
 			(effects
 				(font
@@
 		)
 		(property "Description" "Resistor, small symbol"
-			(at 142.24 127 0)
+			(at 149.86 119.38 0)
 			(effects
 				(font
@@
 	(symbol
 		(lib_id "power:+3.3V")
-		(at 142.24 114.3 0)
+		(at 149.86 111.76 0)
 		(unit 1)
 		(exclude_from_sim no)
@@
 		(fields_autoplaced yes)
 		(property "Reference" "#PWR032"
-			(at 142.24 118.11 0)
+			(at 149.86 115.57 0)
 			(effects
 				(font
@@
 		)
 		(property "Value" "+3.3V"
-			(at 142.24 109.22 0)
+			(at 149.86 106.68 0)
 			(effects
 				(font
@@
 		)
 		(property "Footprint" ""
-			(at 142.24 114.3 0)
+			(at 149.86 111.76 0)
 			(effects
 				(font
@@
 		)
 		(property "Datasheet" ""
-			(at 142.24 114.3 0)
+			(at 149.86 111.76 0)
 			(effects
 				(font
@@
 		)
 		(property "Description" "Power symbol creates a global label with name \"+3.3V\""
-			(at 142.24 114.3 0)
+			(at 149.86 111.76 0)
 			(effects
 				(font
