File: SN65HVD230 .kicad_sch (KiCad schematic)
At the start: 5 parts, among them U1 SN65HVD230

Commit message: layout
Parts:
- added C38: 100n, Capacitor_SMD:C_0402_1005Metric, symbol Device:C_Small
- added D1: NUP2105L, Package_TO_SOT_SMD:SOT-23, symbol Power_Protection:NUP2105L
Connections:
- net 3.3V: now also C38.1
- net can_h: now also D1.2 (K)
- net can_l: now also D1.1 (K)
- net gnd: now also C38.2, D1.3 (A)
