File: foot.kicad_pcb (KiCad board)
At the start: 2 copper layers, 84 parts, among them J1 Conn_01x04_Pin, J2 Conn_01x03_Pin, J3 Conn_01x05_Pin, J4 xt30(2+2), J5 Conn_01x03_Pin, J6 Conn_01x03_Pin, J7 Conn_01x03_Pin, J8 Conn_01x03_Pin, U1 SN65HVD230, U2 AMS1117-3.3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

Commit message: layout
Parts:
- removed R2: 0, Resistor_SMD:R_0603_1608Metric
- added C38: 100n, Capacitor_SMD:C_0402_1005Metric, F.Cu at (75.3, 148.3)
- added D1: NUP2105L, Package_TO_SOT_SMD:SOT-23, F.Cu at (75.2, 161.1)
- added R28: 0, Resistor_SMD:R_0603_1608Metric, F.Cu at (48.2, 149.7)
- added R29: 0, Resistor_SMD:R_0603_1608Metric, F.Cu at (48.2, 151.3)
- added R30: 0, Resistor_SMD:R_0603_1608Metric, F.Cu at (48.2, 152.9)
- C1, C2, C8: value 100n -> 10u; footprint Capacitor_SMD:C_0603_1608Metric -> Capacitor_SMD:C_1206_3216Metric
- C11: value 10u -> 1u
- C3, C9: value 100n -> 1u; footprint Capacitor_SMD:C_0603_1608Metric -> Capacitor_SMD:C_1206_3216Metric
- C4: value 100n -> 10n
- C5, C7: value 100n -> 0.1u; footprint Capacitor_SMD:C_0603_1608Metric -> Capacitor_SMD:C_0402_1005Metric
- R1, R11, R12, R13, R20, R21, R22, R23, R24, R3, R4, R5, R6, R7, R8, R9: footprint Resistor_SMD:R_0603_1608Metric -> Resistor_SMD:R_0402_1005Metric
- R14, R15, R16, R17: value 10k -> 15k; footprint Resistor_SMD:R_0603_1608Metric -> Resistor_SMD:R_0402_1005Metric
- U4: footprint lmr51603:DBV0006A-MFG-IPC_A -> Package_TO_SOT_SMD:TSOT-23-6
- moved R16 95.2 mm to (49.8, 171.4), turned to 90 degrees
- moved R9 92.0 mm to (48.6, 169.4), turned to 90 degrees
- moved C26 89.5 mm to (48.6, 171.4), turned to -90 degrees
- moved J3 86.7 mm to (43.6, 148.2)
- moved C36 82.6 mm to (48.8, 164.9), turned to -90 degrees
- moved R8 74.5 mm to (63.6, 154.8), turned to 90 degrees
- moved C37 73.4 mm to (76.2, 165.0), turned to 90 degrees
- moved FB1 72.3 mm to (56.2, 153.2), turned to 180 degrees
- moved C30 71.9 mm to (66.4, 154.6), turned to -90 degrees
- moved C24 70.5 mm to (47.3, 146.4), turned to 180 degrees
- moved C23 70.3 mm to (49.1, 147.1), turned to -90 degrees
- moved R4 70.1 mm to (59.3, 154.8), turned to 90 degrees
- moved C11 69.8 mm to (52.2, 167.2)
- moved R11 69.5 mm to (64.8, 154.8), turned to 90 degrees
- moved J7 69.4 mm to (45.0, 165.0), turned to -90 degrees
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Connections:
- C10 pad 1: +5V -> +3.3V
- C23 pad 2: Net-(U3-NRST) -> /stm32f446re/NRST
- C24 pad 1: /fx293/adc2 -> Net-(C24-Pad1)
- C25 pad 1: /fx293/adc3 -> Net-(C25-Pad1)
- C26 pad 1: /fx293/adc4 -> Net-(C26-Pad1)
- C27 pad 1: /fx293/adc5 -> Net-(C27-Pad1)
- C5 pad 1: +BATT -> +3.3V
- C7 pad 1: +5V -> +3.3V
- C7 pad 2: /power/fb -> GND
- J3 pad 2: /stm32f446re/TCK -> Net-(J3-Pin_2)
- J3 pad 4: /stm32f446re/TMS -> Net-(J3-Pin_4)
- J3 pad 5: /stm32f446re/NRST -> Net-(J3-Pin_5)
- R1 pad 2: Net-(R1-Pad2) -> /power/fb
- R11 pad 1: Net-(R11-Pad1) -> Net-(C27-Pad1)
- R12 pad 1: Net-(R11-Pad1) -> Net-(C27-Pad1)
- R14 pad 2: /fx293/adc2 -> Net-(C24-Pad1)
- R15 pad 2: /fx293/adc3 -> Net-(C25-Pad1)
- R16 pad 2: /fx293/adc4 -> Net-(C26-Pad1)
- R17 pad 2: /fx293/adc5 -> Net-(C27-Pad1)
- R4 pad 1: Net-(R4-Pad1) -> Net-(C24-Pad1)
- R5 pad 1: Net-(R4-Pad1) -> Net-(C24-Pad1)
- R6 pad 1: Net-(R6-Pad1) -> Net-(C25-Pad1)
- R7 pad 1: Net-(R6-Pad1) -> Net-(C25-Pad1)
- R8 pad 1: Net-(R8-Pad1) -> Net-(C26-Pad1)
- R9 pad 1: Net-(R8-Pad1) -> Net-(C26-Pad1)
- U3 pad 7: Net-(U3-NRST) -> /stm32f446re/NRST
Routing:
- net GND: track 0.00 -> 46.7 mm, vias 0 -> 88
- net Net-(C26-Pad1): track 0.00 -> 31.4 mm, vias 0 -> 2
- net +3.3V: track 0.00 -> 26.4 mm, vias 0 -> 23
- net /can_h: track 0.00 -> 25.7 mm
- net Net-(C25-Pad1): track 0.00 -> 25.3 mm, vias 0 -> 2
- net /stm32f446re/TMS: track 0.00 -> 25.0 mm, vias 0 -> 2
- net /stm32f446re/TCK: track 0.00 -> 24.3 mm, vias 0 -> 2
- net /can_l: track 0.00 -> 24.0 mm
- net Net-(U3-BOOT0): track 0.00 -> 23.6 mm, vias 0 -> 2
- net Net-(C24-Pad1): track 0.00 -> 20.9 mm, vias 0 -> 2
- net /stm32f446re/NRST: track 0.00 -> 20.5 mm, vias 0 -> 3
- net +5V: track 0.00 -> 19.7 mm, vias 0 -> 12
- net Net-(C27-Pad1): track 0.00 -> 17.7 mm, vias 0 -> 2
- net /SN65HVD230/vref: track 0.00 -> 10.2 mm
- net Net-(J3-Pin_5): track 0.00 -> 7.59 mm
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- added copper zone on F.Cu, net +3.3V
- added copper zone on In4.Cu, net +3.3V
- added copper zone on B.Cu, net +5V
- added copper zone on F.Cu, net +5V
- added copper zone on F.Cu, net +BATT
- added copper zone on F.Cu, net /power/sw
- added copper zone on F.Cu, net GND
- added copper zone on In1.Cu, net GND
- added copper zone on In3.Cu, net GND
- added copper zone on F.Cu, net Net-(U4-CB)
Other:
- board outline added: 43 x 46 mm
- copper layers 2 -> 6
