File: power.kicad_sch (KiCad schematic)
At the start: 19 parts, among them U2 AMS1117-3.3, U4 LMR51603YDBVR

Commit message: layout
Parts:
- removed C5, C7: 100n, Capacitor_SMD:C_0603_1608Metric, symbol Device:C_Small
- removed R2: 0, Resistor_SMD:R_0603_1608Metric, symbol Device:R_Small
- C1, C2, C8: value 100n -> 10u; footprint Capacitor_SMD:C_0603_1608Metric -> Capacitor_SMD:C_1206_3216Metric
- C11: value 10u -> 1u
- C3, C9: value 100n -> 1u; footprint Capacitor_SMD:C_0603_1608Metric -> Capacitor_SMD:C_1206_3216Metric
- C4: value 100n -> 10n
- R1, R3: footprint Resistor_SMD:R_0603_1608Metric -> Resistor_SMD:R_0402_1005Metric
- U4: footprint DBV0006A-MFG-IPC_A -> Package_TO_SOT_SMD:TSOT-23-6
Connections:
- net +3.3V: now also C10.1
- net +5V: no longer C10.1
- net fb: now also R1.2
