File: stm32f446re.kicad_sch (KiCad schematic)
At the start: 48 parts, among them J1 Conn_01x04_Pin, J2 Conn_01x03_Pin, J3 Conn_01x05_Pin, U3 STM32F446RETx, Y1 8Mhz

Commit message: layout
Parts:
- added R28, R29, R30: 0, Resistor_SMD:R_0603_1608Metric, symbol Device:R_Small
- R11, R12, R13, R20, R21, R22, R23, R24, R4, R5, R6, R7, R8, R9: footprint Resistor_SMD:R_0603_1608Metric -> Resistor_SMD:R_0402_1005Metric
- R14, R15, R16, R17: value 10k -> 15k; footprint Resistor_SMD:R_0603_1608Metric -> Resistor_SMD:R_0402_1005Metric
Connections:
- net NRST: now also C23.2, U3.7 (NRST), R30.2; no longer J3.5 (Pin_5)
- net TCK: now also R28.2; no longer J3.2 (Pin_2)
- net TMS: now also R29.2; no longer J3.4 (Pin_4)
- net adc2: no longer C24.1, R14.2
- net adc3: no longer C25.1, R15.2
- net adc4: no longer C26.1, R16.2
- net adc5: no longer C27.1, R17.2
- net at R4.1, R5.1: now also C24.1, R14.2
- net at R8.1, R9.1: now also C26.1, R16.2
- net at R6.1, R7.1: now also C25.1, R15.2
- net at R11.1, R12.1: now also C27.1, R17.2
- new net: J3.5 (Pin_5), R30.1
- new net: J3.4 (Pin_4), R29.1
- new net: J3.2 (Pin_2), R28.1
Other:
- moved on the sheet: C24, C25, C26, C27, R12, R14, R15, R16, R17, R5, R7, R9
